Commit message: upload urdfs with stls

File: tests/assets/sample.urdf (robot description, URDF)
Before this commit: robot robot, 13 links, 12 joints
Links:
- link root: geometry collision capsule length=0.2 radius=0.2; collision sphere radius=0.2

Commit message: fix tests

File: tests/assets/sample.urdf (robot description, URDF)
Before this commit: robot robot, 13 links, 12 joints
Links:
- removed link l_elbow1
- removed link l_shoulder1
- removed link l_shoulder2
- removed link l_shoulder3
- removed link l_wrist1
- removed link l_wrist2
- removed link r_elbow1
- removed link r_shoulder1
- removed link r_shoulder2
- removed link r_shoulder3
- removed link r_wrist1
- removed link r_wrist2
- removed link root
- added link base_link, mass 1.0; collision box size=0.2 0.2 0.2; visual box size=0.2 0.2 0.2
- added link forearm_link, mass 0.5; collision cylinder length=0.4 radius=0.05; visual cylinder length=0.4 radius=0.05
- added link teapot_link, mass 0.5; collision mesh filename=teapot.stl; visual mesh filename=teapot.stl
Joints:
- removed joint l_elbow_pitch
- removed joint l_shoulder_pitch
- removed joint l_shoulder_roll
- removed joint l_shoulder_yaw
- removed joint l_wrist_pitch
- removed joint l_wrist_yaw
- removed joint r_elbow_pitch
- removed joint r_shoulder_pitch
- removed joint r_shoulder_roll
- removed joint r_shoulder_yaw
- removed joint r_wrist_pitch
- removed joint r_wrist_yaw
- added joint forearm_teapot_joint: type fixed, parent forearm_link, child teapot_link, origin xyz=0 0.4 0 rpy=0 0 0
- added joint shoulder_joint: type revolute, parent base_link, child forearm_link, origin xyz=0 0.1 0 rpy=0 0 0, axis 0 0 1, limit lower=-1.57 upper=1.57 effort=10.0 velocity=1.0
